File: Hardware/AuxTalon.brd (EAGLE design)
At the start: 70 x 35 mm, 79 parts, among them J1 CONN_AUX_M12_REMOTE, J2 CONN_AUX_M12_REMOTE, J3 CONN_AUX_M12_REMOTE, J4 CONN_TALON_REMOTE, Q1 AO3419, Q2 2N7002, Q3 AO3419, Q4 2N7002, Q5 AO3419, Q6 2N7002, U1 ADS1115, U11 MCP23018QFN, U16 MAX9064, U17 MAX9064, U18 SN74AUP1T87, U19 MAX9064, U2 TXS0102YZP, U20 MAX9064, U21 SN74AUP1T87, U22 MAX9064, U23 MAX9064, U24 SN74AUP1T87, U25 MCP23018QFN, U26 MCP23018QFN, U27 AP1603, U28 74HC4852, U29 SN74AUP1T157DCK, U3 MAX9034TSSOP, U4 INA4180A2, U5 CD4044, U6 SN74HC04, U7 SN74AC08, U8 SIP32431TDFN

Commit message: Preliminary work done on AuxTalon
Parts:
- added C12, C14, C15, C16: 0.1uF, bschulz_passives:C0402
- added C13: 1uF, bschulz_passives:C0805
- added R25, R26, R27: 100k, bschulz_passives:R0402
- added U30: MCP3421A3, bschulz:SOT23-6L
- added U31: PCA9536DFN, bschulz:DFN_8_3X3
- added U32: FXMA2104, bschulz:MLP_12
- C1, C11, C5, C6, C8: device bschulz_passives:C0603 -> bschulz_passives:C0402
- R1, R11, R13, R16, R17, R18, R2, R23, R24, R3, R4, R5, R6, R8, R9: device bschulz_passives:R0603 -> bschulz_passives:R0402
- U2: value TXS0102YZP -> TXS0102DCU; device bschulz:YZP0008 -> bschulz:DCU_(R-PDSO-G8)
- moved R21 356.0 mm to (128.3, 17.8)
- moved R22 356.0 mm to (128.3, 14.0)
- moved U26 356.0 mm to (128.3, 22.9)
- moved C11 345.5 mm to (49.5, 32.1)
- moved U27 336.4 mm to (49.5, 29.2), turned to 180 degrees
- moved L1 333.2 mm to (47.5, 23.4)
- moved C10 329.4 mm to (54.7, 29.2), turned to 270 degrees
- moved C9 318.4 mm to (44.3, 29.2), turned to 270 degrees
- moved R23 317.9 mm to (53.3, -19.1), turned to 90 degrees
- moved R24 317.4 mm to (53.3, -22.9), turned to 90 degrees
- moved U29 308.7 mm to (47.6, -21.1)
- moved U28 303.1 mm to (43.4, -21.1), turned to 180 degrees
- moved S3 297.4 mm to (66.0, 17.8), turned to 270 degrees
- moved R19 281.1 mm to (48.3, 0.00)
- moved R20 281.1 mm to (48.3, -3.81)
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Connections:
- removed net !FAULT4: U5.1, U6.9
- removed net EN4: U5.14, U7.12
- removed net FAULT4: U6.8, U7.13
- removed net LATCH4: U3.14, U5.15
- removed net MOS_CTRL4: U7.11
- removed net SENSE4: U3.13, U4.14
- removed net SENSE4+: U4.12
- removed net SENSE_SWITCHED: U29.6
- removed net VPORT4: U4.13
- new net N$24: U31.1, U32.3
- new net N$25: U31.2, U32.4
- new net N$28: U31.5, U32.5
- new net SWITCHED_SENSE: U29.6, U30.1
- net 3V3: now also C12.1, C13.1, C14.1, C15.1, C16.1, U2.3, U2.6, U30.5, U31.8, U32.2, U32.8; no longer U2.C1, U2.C2
- net 5V: now also R25.2, R26.2, R27.2, U2.7, U32.1; no longer U2.B2
- net GND: now also C12.2, C13.2, C14.2, C15.2, C16.2, U2.2, U30.2, U30.6, U31.4, U32.7; no longer U2.B1
- net MUX_EN: now also R27.1, U32.10; no longer U26.3
- net MUX_SEL0: now also R25.1, U32.12; no longer U26.6
- net MUX_SEL1: now also R26.1, U32.11; no longer U26.7
- net MUX_SEL2: now also U31.3; no longer U26.5
- net SCL: now also U2.5, U30.3, U31.6; no longer U2.D2
- net SCL_HV: now also U2.8; no longer U2.A2
- net SDA: now also U2.4, U30.4, U31.7; no longer U2.D1
- net SDA_HV: now also U2.1; no longer U2.A1
- net VREF: no longer U3.12
Routing:
- net GND: track 0.00 -> 61.0 mm, vias 0 -> 2
- net C11: track 0.00 -> 60.6 mm, vias 0 -> 4
- net C15: track 0.00 -> 59.9 mm, vias 0 -> 4
- net C10: track 0.00 -> 59.7 mm, vias 0 -> 4
- net C0: track 0.00 -> 58.8 mm, vias 0 -> 4
- net C6: track 0.00 -> 58.4 mm, vias 0 -> 4
- net C13: track 0.00 -> 57.8 mm, vias 0 -> 4
- net C5: track 0.00 -> 57.6 mm, vias 0 -> 4
- net C4: track 0.00 -> 57.5 mm, vias 0 -> 4
- net C8: track 0.00 -> 57.5 mm, vias 0 -> 4
- net C7: track 0.00 -> 57.4 mm, vias 0 -> 4
- net C14: track 0.00 -> 57.2 mm, vias 0 -> 4
- net C9: track 0.00 -> 56.9 mm, vias 0 -> 4
- net C2: track 0.00 -> 56.7 mm, vias 0 -> 4
- net C1: track 0.00 -> 56.4 mm, vias 0 -> 4
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- added copper zone on layer 1, net 3V3
- added copper zone on layer 1, net 5V
- added copper zone on layer 1, net GND
- added copper zone on layer 1, net N$17
