File: Hardware/AuxTalon.sch (EAGLE design)
At the start: 79 parts, among them J1 CONN_AUX_M12_REMOTE, J2 CONN_AUX_M12_REMOTE, J3 CONN_AUX_M12_REMOTE, J4 CONN_TALON_REMOTE, Q1 AO3419, Q2 2N7002, Q3 AO3419, Q4 2N7002, Q5 AO3419, Q6 2N7002, U1 ADS1115, U11 MCP23018QFN, U16 MAX9064, U17 MAX9064, U18 SN74AUP1T87, U19 MAX9064, U2 TXS0102YZP, U20 MAX9064, U21 SN74AUP1T87, U22 MAX9064, U23 MAX9064, U24 SN74AUP1T87, U25 MCP23018QFN, U26 MCP23018QFN, U27 AP1603, U28 74HC4852, U29 SN74AUP1T157DCK, U3 MAX9034TSSOP, U4 INA4180A2, U5 CD4044, U6 SN74HC04, U7 SN74AC08, U8 SIP32431TDFN

Commit message: Preliminary work done on AuxTalon
Parts:
- added C12, C14, C15, C16: 0.1uF, bschulz_passives:C-EU0.1UFC0402
- added C13: 1uF, bschulz_passives:C-EU10UFC0805
- added R25, R26, R27: 100k, bschulz_passives:R-EU_100KR0402
- added U30: MCP3421A3, bschulz:MCP3421A3
- added U31: PCA9536DFN, bschulz:PCA9536DFN
- added U32: FXMA2104, bschulz:FXMA2104
- C1, C11, C5, C6, C8: device bschulz_passives:C-EU0.1UFC0603 -> bschulz_passives:C-EU0.1UFC0402
- R1, R11, R2, R24, R6, R8, R9: device bschulz_passives:R-EU_10KR0603 -> bschulz_passives:R-EU_10KR0402
- R13, R16, R17, R18, R3, R4, R5: device bschulz_passives:R-EU_100KR0603 -> bschulz_passives:R-EU_100KR0402
- R23: device bschulz_passives:R-EU_30KR0603 -> bschulz_passives:R-EU_R0402
- U2: value TXS0102YZP -> TXS0102DCU; device bschulz:TXS0102YZP -> bschulz:TXS0102DCU
Connections:
- removed net !FAULT4: U5.Q4, U6.A4
- removed net EN4: U5.R4, U7.A4
- removed net FAULT4: U6.Y4, U7.B4
- removed net LATCH4: U3.OUTD, U5.S4
- removed net MOS_CTRL4: U7.Y4
- removed net SENSE4: U3.IND-, U4.OUT4
- removed net SENSE4+: U4.IN4+
- removed net SENSE_SWITCHED: U29.Y
- removed net VPORT4: U4.IN4-
- new net N$24: U31.P0, U32.A1
- new net N$25: U31.P1, U32.A2
- new net N$28: U31.P3, U32.A3
- new net SWITCHED_SENSE: U29.Y, U30.VIN+
- net 3V3: now also C12.1, C13.1, C14.1, C15.1, C16.1, U30.VDD, U31.VCC, U32.EN, U32.VA
- net 5V: now also R25.2, R26.2, R27.2, U32.VB
- net GND: now also C12.2, C13.2, C14.2, C15.2, C16.2, U30.VIN-, U30.VSS, U31.GND, U32.GND
- net MUX_EN: now also R27.1, U32.B3; no longer U26.GPB3
- net MUX_SEL0: now also R25.1, U32.B1; no longer U26.GPB6
- net MUX_SEL1: now also R26.1, U32.B2; no longer U26.GPB7
- net MUX_SEL2: now also U31.P2; no longer U26.GPB5
- net SCL: now also U30.SCL, U31.SCL
- net SDA: now also U30.SDA, U31.SDA
- net VREF: no longer U3.IND+
