File: Hardware/AuxTalon_LoadSwitch.sch (EAGLE design)
At the start: 89 parts, among them J1 CONN_AUX_M12_REMOTE, J2 CONN_AUX_M12_REMOTE, J3 CONN_AUX_M12_REMOTE, J4 CONN_TALON_REMOTE, U1 ADS1115, U11 MCP23018QFN, U16 MAX9064, U17 MAX9064, U18 SN74AUP1T87, U19 MAX9064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

Commit message: Updated part vals for v1.3
Parts:
- C10, C11, C9: value (none) -> 47nF; device bschulz_passives:C-EUC0402 -> bschulz_passives:C-EU47NFC0402
- C2, C3, C4: value 4.7uF -> 0.1uF; device bschulz_passives:C-EU4.7UFC0805 -> bschulz_passives:C-EU0.1UFC0805
- C21: DIGIKEY (none) -> DNP; MF (none) -> N/A; MPN (none) -> DNP
- L2: DIGIKEY (none) -> 732-4848-1-ND; MF (none) -> Wurth; MPN (none) -> 74438323047
- R10: value 68k -> 100k; device bschulz_passives:R-EU_R0603 -> bschulz_passives:R-EU_100KR0402
- R13, R23, R24: value (none) -> 100k
- R16, R17, R18, R3, R4, R5: value 100k -> 10k; device bschulz_passives:R-EU_100KR0402 -> bschulz_passives:R-EU_10KR0402
- U3, U4, U5: DIGIKEY (none) -> 2156-FPF2006-ND; DISP (none) -> FPF2006; MF (none) -> Fairchild; MPN (none) -> FPF2006
Changed lines of the file:
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@@
 <part name="R1" library="bschulz_passives" deviceset="R-EU_" device="R0402" technology="10K" value="10k"/>
 <part name="R2" library="bschulz_passives" deviceset="R-EU_" device="R0402" technology="10K" value="10k"/>
-<part name="R3" library="bschulz_passives" deviceset="R-EU_" device="R0402" technology="100K" value="100k"/>
-<part name="R4" library="bschulz_passives" deviceset="R-EU_" device="R0402" technology="100K" value="100k"/>
-<part name="R5" library="bschulz_passives" deviceset="R-EU_" device="R0402" technology="100K" value="100k"/>
-<part name="C2" library="bschulz_passives" deviceset="C-EU" device="C0805" technology="4.7UF" value="4.7uF"/>
-<part name="C3" library="bschulz_passives" deviceset="C-EU" device="C0805" technology="4.7UF" value="4.7uF"/>
-<part name="C4" library="bschulz_passives" deviceset="C-EU" device="C0805" technology="4.7UF" value="4.7uF"/>
+<part name="R3" library="bschulz_passives" deviceset="R-EU_" device="R0402" technology="10K" value="10k"/>
+<part name="R4" library="bschulz_passives" deviceset="R-EU_" device="R0402" technology="10K" value="10k"/>
+<part name="R5" library="bschulz_passives" deviceset="R-EU_" device="R0402" technology="10K" value="10k"/>
+<part name="C2" library="bschulz_passives" deviceset="C-EU" device="C0805" technology="0.1UF" value="0.1uF"/>
+<part name="C3" library="bschulz_passives" deviceset="C-EU" device="C0805" technology="0.1UF" value="0.1uF"/>
+<part name="C4" library="bschulz_passives" deviceset="C-EU" device="C0805" technology="0.1UF" value="0.1uF"/>
 <part name="GND6" library="supply1" library_urn="urn:adsk.eagle:library:371" deviceset="GND" device=""/>
 <part name="GND7" library="supply1" library_urn="urn:adsk.eagle:library:371" deviceset="GND" device=""/>
@@
 <part name="U16" library="bschulz" deviceset="MAX906*" device="" technology="4"/>
 <part name="U17" library="bschulz" deviceset="MAX906*" device="" technology="4"/>
-<part name="R16" library="bschulz_passives" deviceset="R-EU_" device="R0402" technology="100K" value="100k"/>
+<part name="R16" library="bschulz_passives" deviceset="R-EU_" device="R0402" technology="10K" value="10k"/>
 <part name="GND33" library="supply1" library_urn="urn:adsk.eagle:library:371" deviceset="GND" device=""/>
 <part name="U18" library="bschulz" deviceset="SN74AUP1T87" device=""/>
@@
 <part name="U19" library="bschulz" deviceset="MAX906*" device="" technology="4"/>
 <part name="U20" library="bschulz" deviceset="MAX906*" device="" technology="4"/>
-<part name="R17" library="bschulz_passives" deviceset="R-EU_" device="R0402" technology="100K" value="100k"/>
+<part name="R17" library="bschulz_passives" deviceset="R-EU_" device="R0402" technology="10K" value="10k"/>
 <part name="GND36" library="supply1" library_urn="urn:adsk.eagle:library:371" deviceset="GND" device=""/>
 <part name="U21" library="bschulz" deviceset="SN74AUP1T87" device=""/>
@@
 <part name="U22" library="bschulz" deviceset="MAX906*" device="" technology="4"/>
 <part name="U23" library="bschulz" deviceset="MAX906*" device="" technology="4"/>
-<part name="R18" library="bschulz_passives" deviceset="R-EU_" device="R0402" technology="100K" value="100k"/>
+<part name="R18" library="bschulz_passives" deviceset="R-EU_" device="R0402" technology="10K" value="10k"/>
 <part name="GND39" library="supply1" library_urn="urn:adsk.eagle:library:371" deviceset="GND" device=""/>
 <part name="U24" library="bschulz" deviceset="SN74AUP1T87" device=""/>
@@
 <part name="C16" library="bschulz_passives" deviceset="C-EU" device="C0402" technology="0.1UF" value="0.1uF"/>
 <part name="GND59" library="supply1" library_urn="urn:adsk.eagle:library:371" deviceset="GND" device=""/>
-<part name="U3" library="bschulz" deviceset="TPS2294*" device="" technology="4"/>
+<part name="U3" library="bschulz" deviceset="TPS2294*" device="" technology="4">
+<attribute name="DIGIKEY" value="2156-FPF2006-ND"/>
+<attribute name="DISP" value="FPF2006"/>
+<attribute name="MF" value="Fairchild"/>
+<attribute name="MPN" value="FPF2006"/>
+</part>
 <part name="C12" library="bschulz_passives" deviceset="C-EU" device="C0805" technology="10UF" value="10uF"/>
 <part name="GND12" library="supply1" library_urn="urn:adsk.eagle:library:371" deviceset="GND" device=""/>
 <part name="GND13" library="supply1" library_urn="urn:adsk.eagle:library:371" deviceset="GND" device=""/>
 <part name="C13" library="bschulz_passives" deviceset="C-EU" device="C0402" technology="0.1UF" value="0.1uF"/>
-<part name="U4" library="bschulz" deviceset="TPS2294*" device="" technology="4"/>
+<part name="U4" library="bschulz" deviceset="TPS2294*" device="" technology="4">
+<attribute name="DIGIKEY" value="2156-FPF2006-ND"/>
+<attribute name="DISP" value="FPF2006"/>
+<attribute name="MF" value="Fairchild"/>
+<attribute name="MPN" value="FPF2006"/>
+</part>
 <part name="C17" library="bschulz_passives" deviceset="C-EU" device="C0805" technology="10UF" value="10uF"/>
 <part name="GND14" library="supply1" library_urn="urn:adsk.eagle:library:371" deviceset="GND" device=""/>
 <part name="GND15" library="supply1" library_urn="urn:adsk.eagle:library:371" deviceset="GND" device=""/>
 <part name="C18" library="bschulz_passives" deviceset="C-EU" device="C0402" technology="0.1UF" value="0.1uF"/>
-<part name="U5" library="bschulz" deviceset="TPS2294*" device="" technology="4"/>
+<part name="U5" library="bschulz" deviceset="TPS2294*" device="" technology="4">
+<attribute name="DIGIKEY" value="2156-FPF2006-ND"/>
+<attribute name="DISP" value="FPF2006"/>
+<attribute name="MF" value="Fairchild"/>
+<attribute name="MPN" value="FPF2006"/>
+</part>
 <part name="C19" library="bschulz_passives" deviceset="C-EU" device="C0805" technology="10UF" value="10uF"/>
 <part name="GND16" library="supply1" library_urn="urn:adsk.eagle:library:371" deviceset="GND" device=""/>
@@
 <part name="C8" library="bschulz_passives" deviceset="C-EU" device="C0805" technology="10UF" value="10uF"/>
 <part name="GND51" library="supply1" library_urn="urn:adsk.eagle:library:371" deviceset="GND" device=""/>
-<part name="R10" library="bschulz_passives" deviceset="R-EU_" device="R0603" value="68k"/>
+<part name="R10" library="bschulz_passives" deviceset="R-EU_" device="R0402" technology="100K" value="100k"/>
 <part name="GND52" library="supply1" library_urn="urn:adsk.eagle:library:371" deviceset="GND" device=""/>
 <part name="GND53" library="supply1" library_urn="urn:adsk.eagle:library:371" deviceset="GND" device=""/>
-<part name="L2" library="bschulz" deviceset="INDUCTOR" device="_MAPI_2.5X2" value="4.7uH"/>
+<part name="L2" library="bschulz" deviceset="INDUCTOR" device="_MAPI_2.5X2" value="4.7uH">
+<attribute name="DIGIKEY" value="732-4848-1-ND"/>
+<attribute name="MF" value="Wurth"/>
+<attribute name="MPN" value="74438323047"/>
+</part>
 <part name="R11" library="bschulz_passives" deviceset="R-EU_" device="R0603" technology="100K" value="100k"/>
 <part name="R12" library="bschulz_passives" deviceset="R-EU_" device="R0603" technology="750K" value="750k"/>
 <part name="GND54" library="supply1" library_urn="urn:adsk.eagle:library:371" deviceset="GND" device=""/>
-<part name="C21" library="bschulz_passives" deviceset="C-EU" device="C0402"/>
+<part name="C21" library="bschulz_passives" deviceset="C-EU" device="C0402">
+<attribute name="DIGIKEY" value="DNP"/>
+<attribute name="MF" value="N/A"/>
+<attribute name="MPN" value="DNP"/>
+</part>
 <part name="C22" library="bschulz_passives" deviceset="C-EU" device="C0805" technology="22UF" value="22uF"/>
 <part name="C23" library="bschulz_passives" deviceset="C-EU" device="C0805" technology="22UF" value="22uF"/>
 <part name="GND55" library="supply1" library_urn="urn:adsk.eagle:library:371" deviceset="GND" device=""/>
-<part name="C9" library="bschulz_passives" deviceset="C-EU" device="C0402"/>
-<part name="C10" library="bschulz_passives" deviceset="C-EU" device="C0402"/>
-<part name="C11" library="bschulz_passives" deviceset="C-EU" device="C0402"/>
-<part name="R13" library="bschulz_passives" deviceset="R-EU_" device="R0402" technology="100K"/>
-<part name="R23" library="bschulz_passives" deviceset="R-EU_" device="R0402" technology="100K"/>
-<part name="R24" library="bschulz_passives" deviceset="R-EU_" device="R0402" technology="100K"/>
+<part name="C9" library="bschulz_passives" deviceset="C-EU" device="C0402" technology="47NF" value="47nF"/>
+<part name="C10" library="bschulz_passives" deviceset="C-EU" device="C0402" technology="47NF" value="47nF"/>
+<part name="C11" library="bschulz_passives" deviceset="C-EU" device="C0402" technology="47NF" value="47nF"/>
+<part name="R13" library="bschulz_passives" deviceset="R-EU_" device="R0402" technology="100K" value="100k"/>
+<part name="R23" library="bschulz_passives" deviceset="R-EU_" device="R0402" technology="100K" value="100k"/>
+<part name="R24" library="bschulz_passives" deviceset="R-EU_" device="R0402" technology="100K" value="100k"/>
 <part name="GND46" library="supply1" library_urn="urn:adsk.eagle:library:371" deviceset="GND" device=""/>
 <part name="GND47" library="supply1" library_urn="urn:adsk.eagle:library:371" deviceset="GND" device=""/>
@@
 <attribute name="NAME" x="127" y="245.11" size="1.778" layer="95" rot="R180"/>
 <attribute name="VALUE" x="127" y="250.19" size="1.778" layer="96" rot="R180"/>
+<attribute name="DIGIKEY" x="121.92" y="246.38" size="1.778" layer="96" rot="R90" display="off"/>
+<attribute name="MF" x="121.92" y="246.38" size="1.778" layer="96" rot="R90" display="off"/>
+<attribute name="MPN" x="121.92" y="246.38" size="1.778" layer="96" rot="R90" display="off"/>
 </instance>
 <instance part="R11" gate="G$1" x="147.32" y="218.44" smashed="yes" rot="R90">
